File: IRInterface/IRInterface.kicad_sch (KiCad schematic)
At the start: 25 parts, among them IC1 THVD1424RGTR, J2 RJHSE5E80, J3 FTSH-105-01-L-DV-007-K, Q1 SFH309, Q2 BC817, Q3 BC807, U1 74LVC1G17, U2 74LVC1G17, U3 STM32G030F6Px

Commit message: Fix review findings
Parts:
- R3: value 180R -> 150R
Connections:
- net +3V3: now also IC1.14 (VCC); no longer IC1.15 (H/~{F})
- net GND: now also IC1.15 (H/~{F}); no longer IC1.14 (VCC)
- no-connect marks 12 -> 14
